Commit message: addressing "port in use" error; ur_hardware_interface does not need to be specific for left/right; fixing rotation error around base in URDF

File: iai_tracy_description/urdf/tracy.urdf.xacro (robot description, xacro)
@@ -44,10 +44,10 @@
         <parent link="left_arm_mount" />
         <child link = "left_base_link" />
-        <origin xyz="0.0 0.0 0.0" rpy="0.0 0.0 0.0" />
+        <origin xyz="0.0 0.0 0.0" rpy="0.0 0.0 ${M_PI}" />
     </joint>
     <joint name="table_right_arm_joint" type="fixed">
         <parent link="right_arm_mount" />
         <child link = "right_base_link" />
-        <origin xyz="0.0 0.0 0.0" rpy="0.0 0.0 ${M_PI}" />
+        <origin xyz="0.0 0.0 0.0" rpy="0.0 0.0 0.0" />
     </joint>
 </robot>

Commit message: add robotiq gripper to URDF

File: iai_tracy_description/urdf/tracy.urdf.xacro (robot description, xacro)
@@ -2,5 +2,5 @@
 <robot xmlns:xacro="http://wiki.ros.org/xacro" name="tracy">
     <xacro:include filename="$(find ur_description)/urdf/inc/ur10e_macro.xacro"/>
-    <!-- <xacro:include filename="$(find robotiq_2f_85_gripper_visualization)/urdf/robotiq_arg2f_85_model.xacro" /> -->
+    <xacro:include filename="$(find robotiq_2f_85_gripper_visualization)/urdf/robotiq_arg2f_85_model_macro.xacro" />
     <xacro:arg name="transmission_hw_interface" default="hardware_interface/PositionJointInterface"/>
     <xacro:arg name="kinematics_config_left" default=""/>
@@ -51,3 +51,15 @@
         <origin xyz="0.0 0.0 0.0" rpy="0.0 0.0 0.0" />
     </joint>
+    <xacro:robotiq_arg2f_85 prefix="left_"/>
+    <xacro:robotiq_arg2f_85 prefix="right_"/>
+    <joint name="right_wrist_gripper_joint" type="fixed">
+        <parent link="right_wrist_3_link" />
+        <child link = "right_robotiq_arg2f_base_link" />
+        <origin xyz="0.0 0.0 0.0" rpy="0.0 0.0 1.57" />
+    </joint>
+    <joint name="left_wrist_gripper_joint" type="fixed">
+        <parent link="left_wrist_3_link" />
+        <child link = "left_robotiq_arg2f_base_link" />
+        <origin xyz="0.0 0.0 0.0" rpy="0.0 0.0 1.57" />
+    </joint>
 </robot>

Commit message: change to beta-robotics fork of robotiq

File: iai_tracy_description/urdf/tracy.urdf.xacro (robot description, xacro)
@@ -2,15 +2,15 @@
 <robot xmlns:xacro="http://wiki.ros.org/xacro" name="tracy">
     <xacro:include filename="$(find ur_description)/urdf/inc/ur10e_macro.xacro"/>
-    <xacro:include filename="$(find robotiq_2f_85_gripper_visualization)/urdf/robotiq_arg2f_85_model_macro.xacro" />
+    <xacro:include filename="$(find robotiq_2f_model)/model/robotiq_2f_85.urdf.xacro" />
     <xacro:arg name="transmission_hw_interface" default="hardware_interface/PositionJointInterface"/>
-    <xacro:arg name="kinematics_config_left" default=""/>
-    <xacro:arg name="kinematics_config_right" default=""/>
+    <xacro:arg name="kinematics_config_left" default="/home/mineumann/work/development/PR2UnrealSimulator/src/iai_tracy/iai_tracy_ur/config/ur10e_controllers_left.yaml"/>
+    <xacro:arg name="kinematics_config_right" default="/home/mineumann/work/development/PR2UnrealSimulator/src/iai_tracy/iai_tracy_ur/config/ur10e_controllers_right.yaml"/>
     <xacro:property name="M_PI" value="3.1415926535897931"/>
-    <link name="world" />
-    <joint name="table_joint" type="fixed">
-        <parent link="world"/>
-        <child link="table"/>
-        <origin xyz="0.0 0.0 0.0" rpy="0.0 0.0 0.0" />
-    </joint>
+    <!-- <link name="world" /> -->
+    <!-- <joint name="table_joint" type="fixed"> -->
+    <!--     <parent link="world"/> -->
+    <!--     <child link="table"/> -->
+    <!--     <origin xyz="0.0 0.0 0.0" rpy="0.0 0.0 0.0" /> -->
+    <!-- </joint> -->
     <link name="table">
         <visual>
@@ -51,15 +51,21 @@
         <origin xyz="0.0 0.0 0.0" rpy="0.0 0.0 0.0" />
     </joint>
-    <xacro:robotiq_arg2f_85 prefix="left_"/>
-    <xacro:robotiq_arg2f_85 prefix="right_"/>
-    <joint name="right_wrist_gripper_joint" type="fixed">
-        <parent link="right_wrist_3_link" />
-        <child link = "right_robotiq_arg2f_base_link" />
-        <origin xyz="0.0 0.0 0.0" rpy="0.0 0.0 1.57" />
-    </joint>
-    <joint name="left_wrist_gripper_joint" type="fixed">
-        <parent link="left_wrist_3_link" />
-        <child link = "left_robotiq_arg2f_base_link" />
-        <origin xyz="0.0 0.0 0.0" rpy="0.0 0.0 1.57" />
-    </joint>
+    <xacro:robotiq_2f_85 parent="left_wrist_3_link"
+                         name="left_gripper">
+      <origin xyz="0 0 0" rpy="0 0 1.5708" />
+    </xacro:robotiq_2f_85>
+    <xacro:robotiq_2f_85 parent="right_wrist_3_link"
+                         name="right_gripper">
+          <origin xyz="0 0 0" rpy="0 0 1.5708" />
+    </xacro:robotiq_2f_85>
+    <!-- <joint name="right_wrist_gripper_joint" type="fixed"> -->
+    <!--     <parent link="right_wrist_3_link" /> -->
+    <!--     <child link = "right_robotiq_arg2f_base_link" /> -->
+    <!--     <origin xyz="0.0 0.0 0.0" rpy="0.0 0.0 1.57" /> -->
+    <!-- </joint> -->
+    <!-- <joint name="left_wrist_gripper_joint" type="fixed"> -->
+    <!--     <parent link="left_wrist_3_link" /> -->
+    <!--     <child link = "left_robotiq_arg2f_base_link" /> -->
+    <!--     <origin xyz="0.0 0.0 0.0" rpy="0.0 0.0 1.57" /> -->
+    <!-- </joint> -->
 </robot>

Commit message: simplified collision model of table in urdf

File: iai_tracy_description/urdf/tracy.urdf.xacro (robot description, xacro)
@@ -21,7 +21,13 @@
         </visual>
         <collision>
-            <origin xyz="0 0 0" rpy="0 0 0"/>
+            <origin xyz="0.59 0 -0.4275" rpy="0 0 0"/>
             <geometry>
-                <mesh filename="package://iai_tracy_description/meshes/tracebot_setup_w_adapter_at_origin.stl" scale="0.001 0.001 0.001"/>
+                <box size="1.18 1.60 0.855" />
+            </geometry>
+        </collision>
+        <collision>
+            <origin xyz="0.135 0 0.125" rpy="0 0 0"/>
+            <geometry>
+                <box size="0.2 0.2 0.25" />
             </geometry>
         </collision>

Commit message: added camera link and pole to tracy urdf

File: iai_tracy_description/urdf/tracy.urdf.xacro (robot description, xacro)
@@ -1,4 +1,7 @@
 <?xml version="1.0"?>
 <robot xmlns:xacro="http://wiki.ros.org/xacro" name="tracy">
+    <material name="grey">
+        <color rgba="0.792156862745098 0.819607843137255 0.933333333333333 1" />
+    </material>
     <xacro:include filename="$(find ur_description)/urdf/inc/ur10e_macro.xacro"/>
     <xacro:include filename="$(find robotiq_2f_85_gripper_visualization)/urdf/robotiq_arg2f_85_model_macro.xacro" />
@@ -15,4 +18,5 @@
     <link name="table">
         <visual>
+            <material name="grey"/>
             <origin xyz="0 0 0" rpy="0 0 0"/>
             <geometry>
@@ -21,4 +25,5 @@
         </visual>
         <collision>
+            <material name="grey"/>
             <origin xyz="0.59 0 -0.4275" rpy="0 0 0"/>
             <geometry>
@@ -27,7 +32,83 @@
         </collision>
         <collision>
-            <origin xyz="0.135 0 0.125" rpy="0 0 0"/>
+            <material name="grey"/>
+            <origin xyz="0.13 0 0.125" rpy="0 0 0"/>
             <geometry>
                 <box size="0.2 0.2 0.25" />
+            </geometry>
+        </collision>
+    </link>
+    <joint name="camera_pole_joint" type="fixed">
+        <parent link="table"/>
+        <child link="camera_pole"/>
+        <origin xyz="0.29 0.0 0.0" rpy="0.0 0.0 0.0" />
+    </joint>
+    <link name="camera_pole">
+        <!-- base -->
+        <visual>
+            <material name="grey"/>
+            <origin xyz="0 0 0.02" rpy="0 0 0"/>
+            <geometry>
+                <box size="0.12 0.455 0.04" />
+            </geometry>
+        </visual>
+        <!-- pole -->
+        <visual>
+            <material name="grey"/>
+            <origin xyz="0 0 0.54" rpy="0 0 0"/>
+            <geometry>
+                <box size="0.04 0.04 1" />
+            </geometry>
+        </visual>
+        <!-- triangle thingy -->
+        <visual>
+            <material name="grey"/>
+            <origin xyz="0 0 0.08" rpy="0 0 0"/>
+            <geometry>
+                <box size="0.04 0.2 0.08" />
+            </geometry>
+        </visual>
+       <!-- base -->
+        <collision>
+            <material name="grey"/>
+            <origin xyz="0 0 0.02" rpy="0 0 0"/>
+            <geometry>
+                <box size="0.12 0.455 0.04" />
+            </geometry>
+        </collision>
+        <!-- pole -->
+        <collision>
+            <material name="grey"/>
+            <origin xyz="0 0 0.54" rpy="0 0 0"/>
+            <geometry>
+                <box size="0.04 0.04 1" />
+            </geometry>
+        </collision>
+        <!-- triangle thingy -->
+        <collision>
+            <material name="grey"/>
+            <origin xyz="0 0 0.08" rpy="0 0 0"/>
+            <geometry>
+                <box size="0.04 0.2 0.08" />
+            </geometry>
+        </collision>
+    </link>
+    <joint name="camera_mount_joint" type="fixed">
+        <parent link="camera_pole"/>
+        <child link="camera_mount"/>
+        <origin xyz="0.0 0.0 0.92" rpy="0.0 0.0 0.0" />
+    </joint>
+    <link name="camera_mount"/>
+   <joint name="camera_link_joint" type="fixed">
+        <parent link="camera_mount"/>
+        <child link="camera_link"/>
+        <origin xyz="0.01 0.0 -0.026" rpy="0.0484812 1.25792843 0.057068" />
+    </joint>
+    <link name="camera_link">
+        <collision>
+            <material name="grey"/>
+            <origin xyz="0 0 0.0" rpy="0 0 0"/>
+            <geometry>
+                <sphere radius="0.05" />
             </geometry>
         </collision>

Commit message: added tool frames

File: iai_tracy_description/urdf/tracy.urdf.xacro (robot description, xacro)
@@ -150,3 +150,15 @@
         <origin xyz="0.0 0.0 0.0" rpy="0.0 0.0 1.57" />
     </joint>
+    <joint name="l_gripper_tool_frame_joint" type="fixed">
+        <parent link="left_robotiq_arg2f_base_link" />
+        <child link = "l_gripper_tool_frame" />
+        <origin xyz="0.0 0.0 0.144" rpy="0.0 0.0 0" />
+    </joint>
+    <link name="l_gripper_tool_frame" />
+    <joint name="r_gripper_tool_frame_joint" type="fixed">
+        <parent link="right_robotiq_arg2f_base_link" />
+        <child link = "r_gripper_tool_frame" />
+        <origin xyz="0.0 0.0 0.144" rpy="0.0 0.0 0" />
+    </joint>
+    <link name="r_gripper_tool_frame" />
 </robot>

Commit message: [camera calibrated URDF] first test

File: iai_tracy_description/urdf/tracy.urdf.xacro (robot description, xacro)
@@ -39,4 +39,15 @@
         </collision>
     </link>
+    <joint name="calibration_point_joint" type="fixed">
+        <parent link="table"/>
+        <child link="calbration_point"/>
+        <origin xyz="0.69 0.0 0.0" rpy="0.0 -${M_PI} 0.0" />
+    </joint>
+    <link name="calibration_point"/>
+    <joint name="calibrated_camera_color_joint" type="fixed">
+        <parent link="calibration_point"/>
+        <child link="calibrated_camera_color_link"/>
+        <origin xyz="0.30369 0.033467 -0.917308" rpy="0.332223 6.26796 4.68759" />
+    </joint>
     <joint name="camera_pole_joint" type="fixed">
         <parent link="table"/>

Commit message: [camera calibrated URDF] bugfixes

File: iai_tracy_description/urdf/tracy.urdf.xacro (robot description, xacro)
@@ -41,5 +41,5 @@
     <joint name="calibration_point_joint" type="fixed">
         <parent link="table"/>
-        <child link="calbration_point"/>
+        <child link="calibration_point"/>
         <origin xyz="0.69 0.0 0.0" rpy="0.0 -${M_PI} 0.0" />
     </joint>
@@ -50,4 +50,5 @@
         <origin xyz="0.30369 0.033467 -0.917308" rpy="0.332223 6.26796 4.68759" />
     </joint>
+    <link name="calibrated_camera_color_link"/>
     <joint name="camera_pole_joint" type="fixed">
         <parent link="table"/>

Commit message: [camera calibrated URDF] added calibrated camera link

File: iai_tracy_description/urdf/tracy.urdf.xacro (robot description, xacro)
@@ -44,11 +44,21 @@
         <origin xyz="0.69 0.0 0.0" rpy="0.0 -${M_PI} 0.0" />
     </joint>
+    <!-- This is the point against which the camera is calibrated-->
     <link name="calibration_point"/>
     <joint name="calibrated_camera_color_joint" type="fixed">
         <parent link="calibration_point"/>
         <child link="calibrated_camera_color_link"/>
-        <origin xyz="0.30369 0.033467 -0.917308" rpy="0.332223 6.26796 4.68759" />
+        <origin xyz="0.303693587994845 0.0334670668154926 -0.917308402826141" rpy="0.33222306128266654 6.2679616550776043 4.6875847864989133" />
     </joint>
+    <!-- This is the link which is calibrated against the calibration point-->
     <link name="calibrated_camera_color_link"/>
+    <joint name="calibrated_camera_joint" type="fixed">
+        <parent link="calibration_point"/>
+        <child link="camera_link"/>
+        <origin xyz="0.303321606346533 0.018473418567805 -0.917080056865077" rpy="3.1882399058998141 5.0449477449563940 3.0726935983898565" />
+    </joint>
+    <!-- This camera link is calculated from an offset of the calibrated link. The offset is calculated from the internal camera model.
+         It is used as an root link for the camera launch file to add all camera links to the world. This includes the camera_color_optical_frame which corresponds to the calibrated frame above-->
+    <link name="camera_link"/>
     <joint name="camera_pole_joint" type="fixed">
         <parent link="table"/>
@@ -114,8 +124,8 @@
    <joint name="camera_link_joint" type="fixed">
         <parent link="camera_mount"/>
-        <child link="camera_link"/>
+        <child link="camera_link2"/>
         <origin xyz="0.01 0.0 -0.026" rpy="0.0484812 1.25792843 0.057068" />
     </joint>
-    <link name="camera_link">
+    <link name="camera_link2">
         <collision>
             <material name="grey"/>

Commit message: manually adjusted camera_link to avoid near-constant shift on object poses

File: iai_tracy_description/urdf/tracy.urdf.xacro (robot description, xacro)
@@ -56,5 +56,7 @@
         <parent link="calibration_point"/>
         <child link="camera_link"/>
-        <origin xyz="0.303321606346533 0.018473418567805 -0.917080056865077" rpy="3.1882399058998141 5.0449477449563940 3.0726935983898565" />
+        <!-- <origin xyz="0.303321606346533 0.018473418567805 -0.917080056865077" rpy="3.1882399058998141 5.0449477449563940 3.0726935983898565" /> -->
+        <!-- Manually adjusted camera_link <-> calibration point offset. Detected markers showed a bit of shift on the y-axis of calibration_point. -->
+        <origin xyz="0.303321606346533 -0.0 -0.917080056865077" rpy="3.1882399058998141 5.0449477449563940 3.0726935983898565" />
     </joint>
     <!-- This camera link is calculated from an offset of the calibrated link. The offset is calculated from the internal camera model.

Commit message: new external camera calibration

File: iai_tracy_description/urdf/tracy.urdf.xacro (robot description, xacro)
@@ -10,9 +10,9 @@
     <xacro:arg name="kinematics_config_right" default=""/>
     <xacro:property name="M_PI" value="3.1415926535897931"/>
-    <link name="world" />
+    <link name="table_base_link" />
     <joint name="table_joint" type="fixed">
-        <parent link="world"/>
+        <parent link="table_base_link"/>
         <child link="table"/>
-        <origin xyz="0.0 0.0 0.0" rpy="0.0 0.0 0.0" />
+        <origin xyz="0.0 0.0 1.0" rpy="0.0 0.0 0.0" />
     </joint>
     <link name="table">
@@ -56,7 +56,9 @@
         <parent link="calibration_point"/>
         <child link="camera_link"/>
-        <!-- <origin xyz="0.303321606346533 0.018473418567805 -0.917080056865077" rpy="3.1882399058998141 5.0449477449563940 3.0726935983898565" /> -->
+        <!--<origin xyz="0.303321606346533 0.018473418567805 -0.917080056865077" rpy="3.1722573891155394 5.0426076904779498 3.0896879692720898" />-->
         <!-- Manually adjusted camera_link <-> calibration point offset. Detected markers showed a bit of shift on the y-axis of calibration_point. -->
-        <origin xyz="0.303321606346533 -0.0 -0.917080056865077" rpy="3.1882399058998141 5.0449477449563940 3.0726935983898565" />
+        <!--<origin xyz="0.303321606346533 -0.0 -0.917080056865077" rpy="3.1722573891155394 5.0426076904779498 3.0896879692720898" />-->
+        <!-- new calibration vlaues from July24-->
+        <origin xyz="0.303763030131944 0.0301312512507701 -0.919836697465432" rpy="3.1931015118480244 5.0413108245636282 3.0939247568977319" />
     </joint>
     <!-- This camera link is calculated from an offset of the calibrated link. The offset is calculated from the internal camera model.

Commit message: adapt tracy urdf to ros2 ur_description package

File: iai_tracy_description/urdf/tracy.urdf.xacro (robot description, xacro)
@@ -4,6 +4,6 @@
         <color rgba="0.792156862745098 0.819607843137255 0.933333333333333 1" />
     </material>
-    <xacro:include filename="$(find ur_description)/urdf/inc/ur10e_macro.xacro"/>
-    <xacro:include filename="$(find robotiq_2f_85_gripper_visualization)/urdf/robotiq_arg2f_85_model_macro.xacro" />
+    <xacro:include filename="$(find ur_description)/urdf/ur_macro.xacro"/>
+    <!-- <xacro:include filename="$(find robotiq_2f_85_gripper_visualization)/urdf/robotiq_arg2f_85_model_macro.xacro" /> -->
     <xacro:arg name="transmission_hw_interface" default="hardware_interface/PositionJointInterface"/>
     <xacro:arg name="kinematics_config_left" default=""/>
@@ -126,17 +126,47 @@
         <origin xyz="0.135 -0.050925 0.173" rpy="1.0472 0.0 0.0" />
     </joint>
-    <xacro:ur10e_robot prefix="left_" transmission_hw_interface="$(arg transmission_hw_interface)" kinematics_parameters_file="$(arg kinematics_config_left)"/>
-    <xacro:ur10e_robot prefix="right_" transmission_hw_interface="$(arg transmission_hw_interface)" kinematics_parameters_file="$(arg kinematics_config_right)"/>
-    <joint name="table_left_arm_joint" type="fixed">
+    <xacro:ur_robot
+     name="ur_left"
+     tf_prefix="left_"
+     parent="left_arm_mount"
+     joint_limits_parameters_file="$(find ur_description)/config/ur10e/joint_limits.yaml"
+     kinematics_parameters_file="$(find ur_description)/config/ur10e/default_kinematics.yaml"
+     physical_parameters_file="$(find ur_description)/config/ur10e/physical_parameters.yaml"
+     visual_parameters_file="$(find ur_description)/config/ur10e/visual_parameters.yaml"
+     safety_limits="false"
+     safety_pos_margin="0.15"
+     safety_k_position="20"
+     force_abs_paths="false"
+     >
+     <origin xyz="0 0 0" rpy="0 0 ${M_PI}" />
+   </xacro:ur_robot>
+    <xacro:ur_robot
+     name="ur_right"
+     tf_prefix="right_"
+     parent="right_arm_mount"
+     joint_limits_parameters_file="$(find ur_description)/config/ur10e/joint_limits.yaml"
+     kinematics_parameters_file="$(find ur_description)/config/ur10e/default_kinematics.yaml"
+     physical_parameters_file="$(find ur_description)/config/ur10e/physical_parameters.yaml"
+     visual_parameters_file="$(find ur_description)/config/ur10e/visual_parameters.yaml"
+     safety_limits="false"
+     safety_pos_margin="0.15"
+     safety_k_position="20"
+     force_abs_paths="false"
+     >
+     <origin xyz="0 0 0" rpy="0 0 0" />
+   </xacro:ur_robot>
+    <!-- <xacro:ur10e_robot prefix="left_" transmission_hw_interface="$(arg transmission_hw_interface)" kinematics_parameters_file="$(arg kinematics_config_left)"/> -->
+    <!-- <xacro:ur10e_robot prefix="right_" transmission_hw_interface="$(arg transmission_hw_interface)" kinematics_parameters_file="$(arg kinematics_config_right)"/> -->
+    <!-- <joint name="table_left_arm_joint" type="fixed">
         <parent link="left_arm_mount" />
         <child link = "left_base_link" />
         <origin xyz="0.0 0.0 0.0" rpy="0.0 0.0 ${M_PI}" />
-    </joint>
-    <joint name="table_right_arm_joint" type="fixed">
+    </joint> -->
+    <!-- <joint name="table_right_arm_joint" type="fixed">
         <parent link="right_arm_mount" />
         <child link = "right_base_link" />
         <origin xyz="0.0 0.0 0.0" rpy="0.0 0.0 0.0" />
-    </joint>
-    <xacro:robotiq_arg2f_85 prefix="left_"/>
+    </joint> -->
+    <!-- <xacro:robotiq_arg2f_85 prefix="left_"/>
     <xacro:robotiq_arg2f_85 prefix="right_"/>
     <joint name="right_wrist_gripper_joint" type="fixed">
@@ -161,4 +191,4 @@
         <origin xyz="0.0 0.0 0.144" rpy="0.0 0.0 0" />
     </joint>
-    <link name="r_gripper_tool_frame" />
+    <link name="r_gripper_tool_frame" /> -->
 </robot>

Commit message: Added gripper and doc

File: iai_tracy_description/urdf/tracy.urdf.xacro (robot description, xacro)
@@ -5,5 +5,6 @@
     </material>
     <xacro:include filename="$(find ur_description)/urdf/ur_macro.xacro"/>
-    <!-- <xacro:include filename="$(find robotiq_2f_85_gripper_visualization)/urdf/robotiq_arg2f_85_model_macro.xacro" /> -->
+    <xacro:include filename="$(find robotiq_description)/urdf/robotiq_2f_85_macro.urdf.xacro"/>
+   <!--<xacro:include filename="$(find robotiq_2f_85_gripper_visualization)/urdf/robotiq_arg2f_85_model_macro.xacro" /> -->
     <xacro:arg name="transmission_hw_interface" default="hardware_interface/PositionJointInterface"/>
     <xacro:arg name="kinematics_config_left" default=""/>
@@ -14,5 +15,5 @@
         <parent link="world"/>
         <child link="table"/>
-        <origin xyz="0.0 0.0 0.0" rpy="0.0 0.0 0.0" />
+        <origin xyz="0.0 0.0 0.88" rpy="0.0 0.0 0.0" />
     </joint>
     <link name="table">
@@ -168,6 +169,11 @@
         <origin xyz="0.0 0.0 0.0" rpy="0.0 0.0 0.0" />
     </joint> -->
+    <xacro:robotiq_gripper name="left_gripper" prefix="left_" parent="left_wrist_3_link">
+       <origin xyz="0.0 0.0 0.0" rpy="0.0 0.0 1.57" />
+    </xacro:robotiq_gripper>
+    <xacro:robotiq_gripper name="right_gripper" prefix="right_" parent="right_wrist_3_link">
+       <origin xyz="0.0 0.0 0.0" rpy="0.0 0.0 1.57" />
+    </xacro:robotiq_gripper>
     <!-- <xacro:robotiq_arg2f_85 prefix="left_"/>
-    <xacro:robotiq_arg2f_85 prefix="right_"/>
     <joint name="right_wrist_gripper_joint" type="fixed">
         <parent link="right_wrist_3_link" />
