Commit message: clean up of ROS1 macros

File: iai_tracy_description/urdf/tracy.urdf.xacro (robot description, xacro)
@@ -157,16 +157,4 @@
      <origin xyz="0 0 0" rpy="0 0 0" />
    </xacro:ur_robot>
-    <!-- <xacro:ur10e_robot prefix="left_" transmission_hw_interface="$(arg transmission_hw_interface)" kinematics_parameters_file="$(arg kinematics_config_left)"/> -->
-    <!-- <xacro:ur10e_robot prefix="right_" transmission_hw_interface="$(arg transmission_hw_interface)" kinematics_parameters_file="$(arg kinematics_config_right)"/> -->
-    <!-- <joint name="table_left_arm_joint" type="fixed">
-        <parent link="left_arm_mount" />
-        <child link = "left_base_link" />
-        <origin xyz="0.0 0.0 0.0" rpy="0.0 0.0 ${M_PI}" />
-    </joint> -->
-    <!-- <joint name="table_right_arm_joint" type="fixed">
-        <parent link="right_arm_mount" />
-        <child link = "right_base_link" />
-        <origin xyz="0.0 0.0 0.0" rpy="0.0 0.0 0.0" />
-    </joint> -->
     <xacro:robotiq_gripper name="left_gripper" prefix="left_" parent="left_wrist_3_link">
        <origin xyz="0.0 0.0 0.0" rpy="0.0 0.0 1.57" />
@@ -175,26 +163,3 @@
        <origin xyz="0.0 0.0 0.0" rpy="0.0 0.0 1.57" />
     </xacro:robotiq_gripper>
-    <!-- <xacro:robotiq_arg2f_85 prefix="left_"/>
-    <joint name="right_wrist_gripper_joint" type="fixed">
-        <parent link="right_wrist_3_link" />
-        <child link = "right_robotiq_arg2f_base_link" />
-        <origin xyz="0.0 0.0 0.0" rpy="0.0 0.0 1.57" />
-    </joint>
-    <joint name="left_wrist_gripper_joint" type="fixed">
-        <parent link="left_wrist_3_link" />
-        <child link = "left_robotiq_arg2f_base_link" />
-        <origin xyz="0.0 0.0 0.0" rpy="0.0 0.0 1.57" />
-    </joint>
-    <joint name="l_gripper_tool_frame_joint" type="fixed">
-        <parent link="left_robotiq_arg2f_base_link" />
-        <child link = "l_gripper_tool_frame" />
-        <origin xyz="0.0 0.0 0.144" rpy="0.0 0.0 0" />
-    </joint>
-    <link name="l_gripper_tool_frame" />
-    <joint name="r_gripper_tool_frame_joint" type="fixed">
-        <parent link="right_robotiq_arg2f_base_link" />
-        <child link = "r_gripper_tool_frame" />
-        <origin xyz="0.0 0.0 0.144" rpy="0.0 0.0 0" />
-    </joint>
-    <link name="r_gripper_tool_frame" /> -->
 </robot>

Commit message: Added toolframes

File: iai_tracy_description/urdf/tracy.urdf.xacro (robot description, xacro)
@@ -163,3 +163,15 @@
        <origin xyz="0.0 0.0 0.0" rpy="0.0 0.0 1.57" />
     </xacro:robotiq_gripper>
+    <joint name="l_gripper_tool_frame_joint" type="fixed">
+        <parent link="left_robotiq_85_base_link" />
+        <child link = "l_gripper_tool_frame" />
+        <origin xyz="0.0 0.0 0.144" rpy="0.0 0.0 0" />
+    </joint>
+    <link name="l_gripper_tool_frame" />
+    <joint name="r_gripper_tool_frame_joint" type="fixed">
+        <parent link="right_robotiq_85_base_link" />
+        <child link = "r_gripper_tool_frame" />
+        <origin xyz="0.0 0.0 0.144" rpy="0.0 0.0 0" />
+    </joint>
+    <link name="r_gripper_tool_frame" />
 </robot>

Commit message: adapted urdf to real robot

File: iai_tracy_description/urdf/tracy.urdf.xacro (robot description, xacro)
@@ -11,7 +11,7 @@
     <xacro:arg name="kinematics_config_right" default=""/>
     <xacro:property name="M_PI" value="3.1415926535897931"/>
-    <link name="world" />
+    <link name="map" />
     <joint name="table_joint" type="fixed">
-        <parent link="world"/>
+        <parent link="map"/>
         <child link="table"/>
         <origin xyz="0.0 0.0 0.88" rpy="0.0 0.0 0.0" />
@@ -158,8 +158,8 @@
    </xacro:ur_robot>
     <xacro:robotiq_gripper name="left_gripper" prefix="left_" parent="left_wrist_3_link">
-       <origin xyz="0.0 0.0 0.0" rpy="0.0 0.0 1.57" />
+       <origin xyz="0.0 0.0 0.0" rpy="0.0 0.0 0.0" />
     </xacro:robotiq_gripper>
     <xacro:robotiq_gripper name="right_gripper" prefix="right_" parent="right_wrist_3_link">
-       <origin xyz="0.0 0.0 0.0" rpy="0.0 0.0 1.57" />
+       <origin xyz="0.0 0.0 0.0" rpy="0.0 0.0 0.0" />
     </xacro:robotiq_gripper>
     <joint name="l_gripper_tool_frame_joint" type="fixed">

Commit message: updated launch for real robot

File: iai_tracy_description/urdf/tracy.urdf.xacro (robot description, xacro)
@@ -127,8 +127,14 @@
         <origin xyz="0.135 -0.050925 0.173" rpy="1.0472 0.0 0.0" />
     </joint>
+    <link name="left_world" />
+    <joint name="left_world_joint" type="fixed">
+        <parent link="left_arm_mount"/>
+        <child link="left_world"/>
+        <origin xyz="0.0 0.0 0.0" rpy="0.0 0.0 ${M_PI}" />
+    </joint>
     <xacro:ur_robot
      name="ur_left"
      tf_prefix="left_"
-     parent="left_arm_mount"
+     parent="left_world"
      joint_limits_parameters_file="$(find ur_description)/config/ur10e/joint_limits.yaml"
      kinematics_parameters_file="$(find ur_description)/config/ur10e/default_kinematics.yaml"
@@ -140,10 +146,16 @@
      force_abs_paths="false"
      >
-     <origin xyz="0 0 0" rpy="0 0 ${M_PI}" />
+     <origin xyz="0 0 0" rpy="0 0 0" />
    </xacro:ur_robot>
+    <link name="right_world" />
+    <joint name="right_world_joint" type="fixed">
+        <parent link="right_arm_mount"/>
+        <child link="right_world"/>
+        <origin xyz="0.0 0.0 0.0" rpy="0.0 0.0 0.0" />
+    </joint>
     <xacro:ur_robot
      name="ur_right"
      tf_prefix="right_"
-     parent="right_arm_mount"
+     parent="right_world"
      joint_limits_parameters_file="$(find ur_description)/config/ur10e/joint_limits.yaml"
      kinematics_parameters_file="$(find ur_description)/config/ur10e/default_kinematics.yaml"

Commit message: Added d435i camera to robot description

File: iai_tracy_description/urdf/tracy.urdf.xacro (robot description, xacro)
@@ -6,4 +6,5 @@
     <xacro:include filename="$(find ur_description)/urdf/ur_macro.xacro"/>
     <xacro:include filename="$(find robotiq_description)/urdf/robotiq_2f_85_macro.urdf.xacro"/>
+    <xacro:include filename="$(find realsense2_description)/urdf/_d435i.urdf.xacro"/>
    <!--<xacro:include filename="$(find robotiq_2f_85_gripper_visualization)/urdf/robotiq_arg2f_85_model_macro.xacro" /> -->
     <xacro:arg name="transmission_hw_interface" default="hardware_interface/PositionJointInterface"/>
@@ -101,18 +102,10 @@
     </joint>
     <link name="camera_mount"/>
-   <joint name="camera_link_joint" type="fixed">
-        <parent link="camera_mount"/>
-        <child link="camera_link"/>
-        <origin xyz="0.01 0.0 -0.026" rpy="0.0484812 1.25792843 0.057068" />
-    </joint>
-    <link name="camera_link">
-        <collision>
-            <material name="grey"/>
-            <origin xyz="0 0 0.0" rpy="0 0 0"/>
-            <geometry>
-                <sphere radius="0.05" />
-            </geometry>
-        </collision>
-    </link>
+    <xacro:sensor_d435i
+      parent="camera_mount"
+      name="camera"
+      use_nominal_extrinsics="true">
+      <origin xyz="0 0 0" rpy="0.0484812 1.25792843 0.057068"/>
+    </xacro:sensor_d435i>
     <link name="left_arm_mount" />
     <joint name="left_arm_joint" type="fixed">

Commit message: recent changes

File: iai_tracy_description/urdf/tracy.urdf.xacro (robot description, xacro)
@@ -8,6 +8,6 @@
    <!--<xacro:include filename="$(find robotiq_2f_85_gripper_visualization)/urdf/robotiq_arg2f_85_model_macro.xacro" /> -->
     <xacro:arg name="transmission_hw_interface" default="hardware_interface/PositionJointInterface"/>
-    <xacro:arg name="kinematics_config_left" default=""/>
-    <xacro:arg name="kinematics_config_right" default=""/>
+    <xacro:arg name="kinematics_config_left" default="$(find ur_description)/config/ur10e/default_kinematics.yaml"/>
+    <xacro:arg name="kinematics_config_right" default="$(find ur_description)/config/ur10e/default_kinematics.yaml"/>
     <xacro:property name="M_PI" value="3.1415926535897931"/>
     <link name="map" />
@@ -104,5 +104,5 @@
         <parent link="camera_mount"/>
         <child link="camera_link"/>
-        <origin xyz="0.01 0.0 -0.026" rpy="0.0484812 1.25792843 0.057068" />
+        <origin xyz="0.01 0.0 -0.026" rpy="0.0484812 1.34792843 0.057068" />
     </joint>
     <link name="camera_link">
@@ -138,5 +138,5 @@
      parent="left_world"
      joint_limits_parameters_file="$(find ur_description)/config/ur10e/joint_limits.yaml"
-     kinematics_parameters_file="$(find ur_description)/config/ur10e/default_kinematics.yaml"
+     kinematics_parameters_file="$(arg kinematics_config_left)"
      physical_parameters_file="$(find ur_description)/config/ur10e/physical_parameters.yaml"
      visual_parameters_file="$(find ur_description)/config/ur10e/visual_parameters.yaml"
@@ -159,5 +159,5 @@
      parent="right_world"
      joint_limits_parameters_file="$(find ur_description)/config/ur10e/joint_limits.yaml"
-     kinematics_parameters_file="$(find ur_description)/config/ur10e/default_kinematics.yaml"
+     kinematics_parameters_file="$(arg kinematics_config_right)"
      physical_parameters_file="$(find ur_description)/config/ur10e/physical_parameters.yaml"
      visual_parameters_file="$(find ur_description)/config/ur10e/visual_parameters.yaml"

Commit message: external calibration => edited camera_mount/camera_pole joint

File: iai_tracy_description/urdf/tracy.urdf.xacro (robot description, xacro)
@@ -98,11 +98,12 @@
         <parent link="camera_pole"/>
         <child link="camera_mount"/>
-        <origin xyz="0.0 0.0 0.92" rpy="0.0 0.0 0.0" />
+	    <!-- <origin xyz="0.0 0.0 0.92" rpy="0.0 0.0 0.0" /> -->
+        <origin xyz="0.012066 -0.036398 0.929310" rpy="-0.031112 -0.077993 -0.011774"/>
     </joint>
     <link name="camera_mount"/>
-   <joint name="camera_link_joint" type="fixed">
+    <joint name="camera_link_joint" type="fixed">
         <parent link="camera_mount"/>
         <child link="camera_link"/>
-        <origin xyz="0.01 0.0 -0.026" rpy="0.0484812 1.34792843 0.057068" />
+	<origin xyz="0.01 0.0 -0.026" rpy="0.0484812 1.34792843 0.057068" />
     </joint>
     <link name="camera_link">

Commit message: URDF change: removed camera_mount; camera_link is now directly connected to camera_pole; calibrated camera_link

File: iai_tracy_description/urdf/tracy.urdf.xacro (robot description, xacro)
@@ -96,15 +96,8 @@
         </collision>
     </link>
-    <joint name="camera_mount_joint" type="fixed">
+    <joint name="camera_link_joint" type="fixed">
         <parent link="camera_pole"/>
-        <child link="camera_mount"/>
-	    <!-- <origin xyz="0.0 0.0 0.92" rpy="0.0 0.0 0.0" /> -->
-        <origin xyz="0.012066 -0.036398 0.929310" rpy="-0.031112 -0.077993 -0.011774"/>
-    </joint>
-    <link name="camera_mount"/>
-    <joint name="camera_link_joint" type="fixed">
-        <parent link="camera_mount"/>
         <child link="camera_link"/>
-	<origin xyz="0.01 0.0 -0.026" rpy="0.0484812 1.34792843 0.057068" />
+        <origin xyz="0.019787 -0.005129 0.922215" rpy="-0.067670 1.375065 -0.073038"/>
     </joint>
     <link name="camera_link">

Commit message: new calibration for camera_link

File: iai_tracy_description/urdf/tracy.urdf.xacro (robot description, xacro)
@@ -97,7 +97,7 @@
     </link>
     <joint name="camera_link_joint" type="fixed">
-        <parent link="camera_pole"/>
+        <parent link="table"/>
         <child link="camera_link"/>
-        <origin xyz="0.019787 -0.005129 0.922215" rpy="-0.067670 1.375065 -0.073038"/>
+        <origin xyz="0.410542 -0.015143 0.932933" rpy="-0.046277 1.378820 -0.050299"/>
     </joint>
     <link name="camera_link">
