Commit message: add gripper adapter to tracy urdf

File: iai_tracy_description/urdf/tracy.urdf.xacro (robot description, xacro)
@@ -12,4 +12,29 @@
     <xacro:arg name="kinematics_config_right" default="$(find ur_description)/config/ur10e/default_kinematics.yaml"/>
     <xacro:property name="M_PI" value="3.1415926535897931"/>
+    <xacro:property name="gripper_coupler_length" value="0.03"/>
+    <xacro:property name="gripper_coupler_radius" value="0.0375"/>
+    <xacro:macro name="gripper_coupler" params="prefix parent">
+        <joint name="${prefix}gripper_coupler_joint" type="fixed">
+            <parent link="${parent}"/>
+            <child link="${prefix}gripper_coupler_link"/>
+            <origin xyz="0 0 0" rpy="0 0 0"/>
+        </joint>
+        <link name="${prefix}gripper_coupler_link">
+            <visual>
+                <origin xyz="0 0 ${gripper_coupler_length / 2}" rpy="0 0 0"/>
+                <geometry>
+                    <cylinder radius="${gripper_coupler_radius}" length="${gripper_coupler_length}"/>
+                </geometry>
+                <material name="coupler_black">
+                    <color rgba="0.1 0.1 0.1 1"/>
+                </material>
+            </visual>
+            <inertial>
+                <origin xyz="0 0 ${gripper_coupler_length / 2}" rpy="0 0 0"/>
+                <mass value="0.2"/>
+                <inertia ixx="0.00011" ixy="0.0" ixz="0.0" iyy="0.00011" iyz="0.0" izz="0.00014"/>
+            </inertial>
+        </link>
+    </xacro:macro>
     <link name="map" />
     <joint name="table_joint" type="fixed">
@@ -99,5 +124,6 @@
         <parent link="table"/>
         <child link="camera_link"/>
-        <origin xyz="0.410542 -0.015143 0.932933" rpy="-0.046277 1.378820 -0.050299"/>
+        <!-- <origin xyz="0.410542 -0.015143 0.932933" rpy="-0.046277 1.378820 -0.050299"/>: -->
+        <origin xyz="0.403282 0.019766 0.881559" rpy="-0.016644 1.135460 -0.005690"/>
     </joint>
     <link name="camera_link">
@@ -172,9 +198,11 @@
      <origin xyz="0 0 0" rpy="0 0 0" />
    </xacro:ur_robot>
-    <xacro:robotiq_gripper name="left_gripper" prefix="left_" parent="left_wrist_3_link">
-       <origin xyz="0.0 0.0 0.0" rpy="0.0 0.0 0.0" />
+    <xacro:gripper_coupler prefix="left_" parent="left_wrist_3_link"/>
+    <xacro:gripper_coupler prefix="right_" parent="right_wrist_3_link"/>
+    <xacro:robotiq_gripper name="left_gripper" prefix="left_" parent="left_gripper_coupler_link">
+       <origin xyz="0.0 0.0 ${gripper_coupler_length}" rpy="0.0 0.0 0.0" />
     </xacro:robotiq_gripper>
-    <xacro:robotiq_gripper name="right_gripper" prefix="right_" parent="right_wrist_3_link">
-       <origin xyz="0.0 0.0 0.0" rpy="0.0 0.0 0.0" />
+    <xacro:robotiq_gripper name="right_gripper" prefix="right_" parent="right_gripper_coupler_link">
+       <origin xyz="0.0 0.0 ${gripper_coupler_length}" rpy="0.0 0.0 0.0" />
     </xacro:robotiq_gripper>
     <joint name="l_gripper_tool_frame_joint" type="fixed">
